Commit message: Setup ros code for visualising model and setting joints. Tweaked model to remove closed loops.

File: catkin_ws/src/gripperv4/urdf/gripperv4.urdf (robot description, URDF)
Before this commit: robot gripperv4, 13 links, 14 joints
Links:
- removed link l_link21
- removed link r_link21
- added link base_link_actual, mass 0.009061016616131982; collision mesh filename=package://gripperv4/assets/base_link.stl scale=0.001 0.001 0.001; visual mesh filename=package://gripperv4/assets/base_link.stl scale=0.001 0.001 0.001
- link base_link: mass 0.009061016616131982 -> None; geometry 
- link gripper_mount1: geometry collision mesh filename=package://gripperv4/assets/gripper_mount1.stl scale=0.001 0.001 0.001; visual mesh filename=package://gripperv4/assets/gripper_mount1.stl scale=0.001 0.001 0.001
- link l_link11: geometry collision mesh filename=package://gripperv4/assets/l_link11.stl scale=0.001 0.001 0.001; visual mesh filename=package://gripperv4/assets/l_link11.stl scale=0.001 0.001 0.001
- link l_link31: geometry collision mesh filename=package://gripperv4/assets/l_link31.stl scale=0.001 0.001 0.001; visual mesh filename=package://gripperv4/assets/l_link31.stl scale=0.001 0.001 0.001
- link l_servo1: geometry collision mesh filename=package://gripperv4/assets/l_servo1.stl scale=0.001 0.001 0.001; visual mesh filename=package://gripperv4/assets/l_servo1.stl scale=0.001 0.001 0.001
- link r_link11: geometry collision mesh filename=package://gripperv4/assets/r_link11.stl scale=0.001 0.001 0.001; visual mesh filename=package://gripperv4/assets/r_link11.stl scale=0.001 0.001 0.001
- link r_link31: geometry collision mesh filename=package://gripperv4/assets/r_link31.stl scale=0.001 0.001 0.001; visual mesh filename=package://gripperv4/assets/r_link31.stl scale=0.001 0.001 0.001
- link r_servo1: geometry collision mesh filename=package://gripperv4/assets/r_servo1.stl scale=0.001 0.001 0.001; visual mesh filename=package://gripperv4/assets/r_servo1.stl scale=0.001 0.001 0.001
- link roll2yaw_mount1: geometry collision mesh filename=package://gripperv4/assets/roll2yaw_mount1.stl scale=0.001 0.001 0.001; visual mesh filename=package://gripperv4/assets/roll2yaw_mount1.stl scale=0.001 0.001 0.001
- link roll_servo1: geometry collision mesh filename=package://gripperv4/assets/roll_servo1.stl scale=0.001 0.001 0.001; visual mesh filename=package://gripperv4/assets/roll_servo1.stl scale=0.001 0.001 0.001
- link yaw_servo1: geometry collision mesh filename=package://gripperv4/assets/yaw_servo1.stl scale=0.001 0.001 0.001; visual mesh filename=package://gripperv4/assets/yaw_servo1.stl scale=0.001 0.001 0.001
Joints:
- removed joint Rev100
- removed joint Rev101
- removed joint Rev96
- removed joint Rev97
- added joint dummy_link: type fixed, parent base_link, child base_link_actual, origin xyz=0 0 0 rpy=0 0 0

Commit message: Added new URDF with hopefully correct joints

File: catkin_ws/src/gripperv4/urdf/gripperv4.urdf (robot description, URDF)
Before this commit: robot gripperv4, 12 links, 11 joints
Links:
- removed link base_link_actual
- removed link l_servo1
- removed link r_servo1
- removed link roll2yaw_mount1
- removed link roll_servo1
- removed link yaw_servo1
- added link roll_yaw_servo1, mass 0.6469480906726006; collision mesh filename=meshes/roll_yaw_servo1.stl scale=0.001 0.001 0.001; visual mesh filename=meshes/roll_yaw_servo1.stl scale=0.001 0.001 0.001
- link base_link: mass None -> 0.009061016616131982; geometry collision mesh filename=meshes/base_link.stl scale=0.001 0.001 0.001; visual mesh filename=meshes/base_link.stl scale=0.001 0.001 0.001
- link gripper_mount1: mass 0.03378268770833562 -> 0.6707222526282031; geometry collision mesh filename=meshes/gripper_mount1.stl scale=0.001 0.001 0.001; visual mesh filename=meshes/gripper_mount1.stl scale=0.001 0.001 0.001
- link l_link11: geometry collision mesh filename=meshes/l_link11.stl scale=0.001 0.001 0.001; visual mesh filename=meshes/l_link11.stl scale=0.001 0.001 0.001
- link l_link31: geometry collision mesh filename=meshes/l_link31.stl scale=0.001 0.001 0.001; visual mesh filename=meshes/l_link31.stl scale=0.001 0.001 0.001
- link r_link11: geometry collision mesh filename=meshes/r_link11.stl scale=0.001 0.001 0.001; visual mesh filename=meshes/r_link11.stl scale=0.001 0.001 0.001
- link r_link31: geometry collision mesh filename=meshes/r_link31.stl scale=0.001 0.001 0.001; visual mesh filename=meshes/r_link31.stl scale=0.001 0.001 0.001
Joints:
- removed joint Rev88
- removed joint Rev91
- removed joint Rev94
- removed joint Rev95
- removed joint Rev98
- removed joint Rev99
- removed joint Rigid89
- removed joint Rigid90
- removed joint Rigid92
- removed joint Rigid93
- removed joint dummy_link
- added joint Rev_base: type continuous, parent base_link, child roll_yaw_servo1, origin xyz=0.016 -0.095 -0.0374 rpy=0 0 0, axis 0.0 0.0 1.0
- added joint Rev_left: type continuous, parent gripper_mount1, child l_link11, origin xyz=-0.016 0.0466 0.0166 rpy=0 0 0, axis 0.0 0.0 1.0
- added joint Rev_left_finger: type continuous, parent l_link11, child l_link31, origin xyz=0.0 0.05 0.0014 rpy=0 0 0, axis 0.0 0.0 -1.0
- added joint Rev_right: type continuous, parent gripper_mount1, child r_link11, origin xyz=0.016 0.0466 0.0166 rpy=0 0 0, axis 0.0 0.0 1.0
- added joint Rev_right_finger: type continuous, parent r_link11, child r_link31, origin xyz=0.0 0.05 0.0014 rpy=0 0 0, axis 0.0 0.0 1.0
- added joint Rev_roll: type continuous, parent roll_yaw_servo1, child gripper_mount1, origin xyz=0.0 0.0484 0.0164 rpy=0 0 0, axis 0.0 1.0 -0.0

Commit message: Visualisation successful in RViz with updated joints

File: catkin_ws/src/gripperv4/urdf/gripperv4.urdf (robot description, URDF)
Before this commit: robot gripperv4, 7 links, 6 joints
Links:
- added link base_link_actual, mass 0.009061016616131982; collision mesh filename=package://gripperv4/assets/base_link.stl scale=0.001 0.001 0.001; visual mesh filename=package://gripperv4/assets/base_link.stl scale=0.001 0.001 0.001
- link base_link: mass 0.009061016616131982 -> None; geometry 
- link gripper_mount1: geometry collision mesh filename=package://gripperv4/assets/gripper_mount1.stl scale=0.001 0.001 0.001; visual mesh filename=package://gripperv4/assets/gripper_mount1.stl scale=0.001 0.001 0.001
- link l_link11: geometry collision mesh filename=package://gripperv4/assets/l_link11.stl scale=0.001 0.001 0.001; visual mesh filename=package://gripperv4/assets/l_link11.stl scale=0.001 0.001 0.001
- link l_link31: geometry collision mesh filename=package://gripperv4/assets/l_link31.stl scale=0.001 0.001 0.001; visual mesh filename=package://gripperv4/assets/l_link31.stl scale=0.001 0.001 0.001
- link r_link11: geometry collision mesh filename=package://gripperv4/assets/r_link11.stl scale=0.001 0.001 0.001; visual mesh filename=package://gripperv4/assets/r_link11.stl scale=0.001 0.001 0.001
- link r_link31: geometry collision mesh filename=package://gripperv4/assets/r_link31.stl scale=0.001 0.001 0.001; visual mesh filename=package://gripperv4/assets/r_link31.stl scale=0.001 0.001 0.001
- link roll_yaw_servo1: geometry collision mesh filename=package://gripperv4/assets/roll_yaw_servo1.stl scale=0.001 0.001 0.001; visual mesh filename=package://gripperv4/assets/roll_yaw_servo1.stl scale=0.001 0.001 0.001
Joints:
- added joint dummy_link: type fixed, parent base_link, child base_link_actual, origin xyz=0 0 0 rpy=0 0 0

Commit message: Updated with new design and added code to control DYNAMIXELs individually

File: catkin_ws/src/gripperv4/urdf/gripperv4.urdf (robot description, URDF)
Before this commit: robot gripperv4, 8 links, 7 joints
Links:
- removed link l_link31
- removed link r_link31
- added link l_finger1, mass 0.023712538812289255; collision mesh filename=package://gripperv4/assets/l_finger1.stl scale=0.001 0.001 0.001; visual mesh filename=package://gripperv4/assets/l_finger1.stl scale=0.001 0.001 0.001
- added link l_link21, mass 0.00386409068463368; collision mesh filename=package://gripperv4/assets/l_link21.stl scale=0.001 0.001 0.001; visual mesh filename=package://gripperv4/assets/l_link21.stl scale=0.001 0.001 0.001
- added link pitch_mount1, mass 0.08039663104912372; collision mesh filename=package://gripperv4/assets/pitch_mount1.stl scale=0.001 0.001 0.001; visual mesh filename=package://gripperv4/assets/pitch_mount1.stl scale=0.001 0.001 0.001
- added link r_finger1, mass 0.023712538812289255; collision mesh filename=package://gripperv4/assets/r_finger1.stl scale=0.001 0.001 0.001; visual mesh filename=package://gripperv4/assets/r_finger1.stl scale=0.001 0.001 0.001
- added link r_link21, mass 0.0038640906846336806; collision mesh filename=package://gripperv4/assets/r_link21.stl scale=0.001 0.001 0.001; visual mesh filename=package://gripperv4/assets/r_link21.stl scale=0.001 0.001 0.001
- link base_link_actual: mass 0.009061016616131982 -> 0.9490572232520995
- link gripper_mount1: mass 0.6707222526282031 -> 0.6706735500880907
- link l_link11: mass 0.014672073181914151 -> 0.013747989643093032
- link r_link11: mass 0.014672069251285016 -> 0.01374798583124482
Joints:
- removed joint Rev_base
- added joint Rev_left_support: type continuous, parent gripper_mount1, child l_link21, origin xyz=-0.039617 0.0281 0.006 rpy=0 0 0, axis -0.0 0.0 -1.0
- added joint Rev_pitch: type continuous, parent base_link, child pitch_mount1, origin xyz=0.0354 -0.063124 0.021 rpy=0 0 0, axis 1.0 0.0 0.0
- added joint Rev_right_support: type continuous, parent gripper_mount1, child r_link21, origin xyz=0.039617 0.0281 0.006 rpy=0 0 0, axis 0.0 -0.0 1.0
- added joint Rev_yaw: type continuous, parent pitch_mount1, child roll_yaw_servo1, origin xyz=-0.035383 0.063124 0.0184 rpy=0 0 0, axis 0.0 0.0 1.0
- joint Rev_left: axis 0.0 0.0 1.0 -> 0.0 -0.0 1.0; origin xyz=-0.016 0.0466 0.0166 rpy=0 0 0 -> xyz=-0.016 0.0466 0.0164 rpy=0 0 0
- joint Rev_left_finger: axis 0.0 0.0 -1.0 -> -0.0 0.0 -1.0; child l_link31 -> l_finger1; origin xyz=0.0 0.05 0.0014 rpy=0 0 0 -> xyz=0.0 0.035 0.0016 rpy=0 0 0
- joint Rev_right: axis 0.0 0.0 1.0 -> 0.0 -0.0 1.0; origin xyz=0.016 0.0466 0.0166 rpy=0 0 0 -> xyz=0.016 0.0466 0.0164 rpy=0 0 0
- joint Rev_right_finger: axis 0.0 0.0 1.0 -> 0.0 -0.0 1.0; child r_link31 -> r_finger1; origin xyz=0.0 0.05 0.0014 rpy=0 0 0 -> xyz=0.0 0.035 0.0016 rpy=0 0 0
- joint Rev_roll: origin xyz=0.0 0.0484 0.0164 rpy=0 0 0 -> xyz=0.0 0.0484 -0.0184 rpy=0 0 0
